Commit message: first commit

File: source/yam_simulator_2/yam_simulator_2/assets/yam/yam.urdf (robot description, URDF)
Before this commit: robot yam_v0, 7 links, 6 joints
Links:
- added link gripper_base
- added link left_finger
- added link right_finger
- link base_link: geometry collision mesh filename=assets/base_link_collision.stl; visual mesh filename=assets/base_link_visual.stl
- link link_1: geometry collision mesh filename=assets/link_1_collision.stl; visual mesh filename=assets/link_1_visual.stl
- link link_2: geometry collision mesh filename=assets/link_2_collision.stl; visual mesh filename=assets/link_2_visual.stl
- link link_3: geometry collision mesh filename=assets/link_3_collision.stl; visual mesh filename=assets/link_3_visual.stl
- link link_4: geometry collision mesh filename=assets/link_4_collision.stl; visual mesh filename=assets/link_4_visual.stl
- link link_5: geometry collision mesh filename=assets/link_5_collision.stl; visual mesh filename=assets/link_5_visual.stl
- link link_6: geometry collision mesh filename=assets/link_6_collision.stl; visual mesh filename=assets/link_6_visual.stl
Joints:
- added joint gripper_mount: type fixed, parent link_6, child gripper_base, origin xyz=0 0 0.10 rpy=0 0 0
- added joint left_finger_joint: type prismatic, parent gripper_base, child left_finger, origin xyz=0 0 0 rpy=0 0 0, axis 1 0 0, limit lower=0.0 upper=0.04 effort=50 velocity=0.2
- added joint right_finger_joint: type prismatic, parent gripper_base, child right_finger, origin xyz=0 0 0 rpy=0 0 0, axis 1 0 0, limit lower=0.0 upper=0.04 effort=50 velocity=0.2, mimic joint=left_finger_joint multiplier=-1 offset=0
